Commit message: [Udpate Oscar]

File: lukas_ws/src/lukas_control/description/lukas.xacro.urdf (robot description, URDF)
Before this commit: robot two_link_arm_xz, 3 links, 2 joints
Links:
- removed link base_link
- removed link link1
- removed link link2
Joints:
- removed joint joint1
- removed joint joint2
